File: pdtrigger.kicad_sch (KiCad schematic)
At the start: 83 parts, among them J1 Conn_01x04_Pin, J2 USB_C_Receptacle_USB2.0_16P, J3 Conn_01x02_Pin, Q1 DMP3098LSD-13, Q3 NMOS, SW1 SW_SPDT, SW2 SW_Push, U1 STM32F401RBT6, U2 CYPD3177-24LQXQ, U3 TERM_BLK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

Commit message: Prettier schematic
Other:
- note added: "3V3 Buck Converter"
- note added: "Debugging Button/LEDs"
- note added: "Microcontroller"
- note added: "PDO Select"
- moved on the sheet: C1, C10, C11, C12, C13, C14, C15, C16, C17, C18, C19, C2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

Commit message: Changed as per design review
Parts:
- added D8, D9: USBLC6-2P6, libs:SOT-666-6_L1.6-W1.2-P0.50-LS1.6-BR, symbol libs:USBLC6-2P6
Connections:
- net CC1: now also D9.3 (I/O2), D9.4 (I/O2)
- net CC2: now also D9.1 (I/O1), D9.6 (I/O1)
- net GND: now also D8.2 (GND), D9.2 (GND)
- net USB_D+: now also D8.1 (I/O1), D8.6 (I/O1)
- net USB_D-: now also D8.3 (I/O2), D8.4 (I/O2)
- net VBUS: now also D9.5 (VBUS)
- no-connect marks 34 -> 35
Other:
- note removed: "With STM32F401 for power profile selection"
- moved on the sheet: C12, C13, C14, C15, C16, C17, C18, C19, C20, J2, J3, Q1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
